Commit message: Complete overhaul of the 2F85 URDF.

File: models/UR5_2F85.urdf (robot description, URDF)
Before this commit: robot starsthing, 22 links, 21 joints
Links:
- removed link tool0
- added link tcp
- link gripper_base: mass 0.5 -> 0.60831; geometry collision mesh filename=package://Robotiq_2F85/meshes/base.STL; visual mesh filename=package://Robotiq_2F85/meshes/base.STL
- link gripper_left_coupler: mass 0.1 -> 0.0273093985570947; geometry collision mesh filename=package://Robotiq_2F85/meshes/left_coupler.STL; visual mesh filename=package://Robotiq_2F85/meshes/left_coupler.STL
- link gripper_left_driver: mass 0.1 -> 0.0184906489414316; geometry collision mesh filename=package://Robotiq_2F85/meshes/left_driver.STL; visual mesh filename=package://Robotiq_2F85/meshes/left_driver.STL
- link gripper_left_follower: mass 0.1 -> 0.0195548943464751; geometry collision mesh filename=package://Robotiq_2F85/meshes/left_follower.STL; visual mesh filename=package://Robotiq_2F85/meshes/left_follower.STL
- link gripper_left_pad: mass 0.1 -> 0.0112846745192961; geometry collision mesh filename=package://Robotiq_2F85/meshes/left_pad.STL; visual mesh filename=package://Robotiq_2F85/meshes/left_pad.STL
- link gripper_left_spring_link: mass 0.1 -> 0.0299513316731757; geometry collision mesh filename=package://Robotiq_2F85/meshes/left_spring_link.STL; visual mesh filename=package://Robotiq_2F85/meshes/left_spring_link.STL
- link gripper_right_coupler: mass 0.1 -> 0.0273093985570947; geometry collision mesh filename=package://Robotiq_2F85/meshes/right_coupler.STL; visual mesh filename=package://Robotiq_2F85/meshes/right_coupler.STL
- link gripper_right_driver: mass 0.1 -> 0.0184906489409923; geometry collision mesh filename=package://Robotiq_2F85/meshes/right_driver.STL; visual mesh filename=package://Robotiq_2F85/meshes/right_driver.STL
- link gripper_right_follower: mass 0.1 -> 0.0195548943464751; geometry collision mesh filename=package://Robotiq_2F85/meshes/right_follower.STL; visual mesh filename=package://Robotiq_2F85/meshes/right_follower.STL
- link gripper_right_pad: mass 0.1 -> 0.0112846745192962; geometry collision mesh filename=package://Robotiq_2F85/meshes/right_pad.STL; visual mesh filename=package://Robotiq_2F85/meshes/right_pad.STL
- link gripper_right_spring_link: mass 0.1 -> 0.029951; geometry collision mesh filename=package://Robotiq_2F85/meshes/right_spring_link.STL; visual mesh filename=package://Robotiq_2F85/meshes/right_spring_link.STL
Joints:
- removed joint ee_link-tool0
- added joint tool_center_point: type fixed, parent gripper_base, child tcp, origin xyz=0 -0.14948 0 rpy=1.5707963267948966 1.5707963267948966 0
- joint ee_link_gripper_base_joint: origin xyz=0 0 0 rpy=0 1.5707963267948966 0 -> xyz=0 0 0 rpy=0 0 1.5707963267948966
- joint gripper_left_coupler_joint: axis 1 0 0 -> 0 0 1; limit lower=-2.9670591111111113 upper=2.9670591111111113 effort=176 velocity=1.919861777777778 -> lower=0.13 upper=0.79 effort=0 velocity=0; origin xyz=0 0.0315 -0.0041 rpy=0 0 0 -> xyz=0.031486 -0.0040855 0 rpy=3.1416 0 -3.1416
- joint gripper_left_driver_joint: axis 1 0 0 -> 0 0 1; limit lower=0.0 upper=0.8726644444444445 effort=176 velocity=1.919861777777778 -> lower=-3.1416 upper=3.1416 effort=150 velocity=0; origin xyz=0 -0.0306011 0.054904 rpy=0 0 3.141592653589793 -> xyz=-0.030601 -0.054792 0 rpy=0 0 -3.1245
- joint gripper_left_follower_joint: axis 1 0 0 -> 0 0 1; limit lower=-2.9670591111111113 upper=2.9670591111111113 effort=176 velocity=1.919861777777778 -> lower=-3.1416 upper=3.1416 effort=0 velocity=0; origin xyz=0 0.0061 0.0471 rpy=0 0 0 -> xyz=-0.0061148 0.047125 0 rpy=0 0 0.017192
- joint gripper_left_pad_joint: axis (none) -> 0 -1 0; limit (none) -> lower=0 upper=0.003 effort=5 velocity=0.1; origin (none) -> xyz=0.018903 0.032265 0 rpy=0 0 -1.5708; type fixed -> prismatic
- joint gripper_left_spring_link_joint: axis 1 0 0 -> 0 0 1; limit lower=-2.9670591111111113 upper=2.9670591111111113 effort=176 velocity=1.919861777777778 -> lower=-0.7854 upper=0 effort=0 velocity=0; origin xyz=0 -0.012 0.0614 rpy=0 0 3.141592653589793 -> xyz=-0.0127 -0.061307 0 rpy=3.1416 0 -0.70092
- joint gripper_right_coupler_joint: axis 1 0 0 -> 0 0 -1; limit lower=-2.9670591111111113 upper=2.9670591111111113 effort=176 velocity=1.919861777777778 -> lower=0.13 upper=0.79 effort=0 velocity=0; origin xyz=0 0.0315 -0.0041 rpy=0 0 0 -> xyz=0.031486 -0.0040855 0 rpy=0 0 -0.25804
- joint gripper_right_driver_joint: axis 1 0 0 -> 0 0 1; limit lower=0.0 upper=0.8726644444444445 effort=176 velocity=1.919861777777778 -> lower=-3.1416 upper=3.1416 effort=150 velocity=0; origin xyz=0 0.0306011 0.054904 rpy=0 0 0 -> xyz=0.030601 -0.054792 0 rpy=3.1416 0 -0.019735
- joint gripper_right_follower_joint: axis 1 0 0 -> 0 0 1; limit lower=-2.9670591111111113 upper=2.9670591111111113 effort=176 velocity=1.919861777777778 -> lower=-3.1416 upper=3.1416 effort=0 velocity=0; origin xyz=0 0.0061 0.0471 rpy=0 0 0 -> xyz=-0.0061148 0.047125 0 rpy=3.1416 0 -2.9033
- joint gripper_right_pad_joint: axis (none) -> 0 1 0; limit (none) -> lower=0 upper=0.003 effort=5 velocity=0.1; origin (none) -> xyz=0.024903 0.032264 0 rpy=3.1416 0 -1.5708
- joint gripper_right_spring_link_joint: axis 1 0 0 -> 0 0 1; limit lower=-2.9670591111111113 upper=2.9670591111111113 effort=176 velocity=1.919861777777778 -> lower=0 upper=0.7854 effort=0 velocity=0; origin xyz=0 0.012 0.0614 rpy=0 0 0 -> xyz=0.0127 -0.061307 0 rpy=3.1416 0 0.6983

File: models/UR5_2F85_BuildURDF.xacro (robot description, xacro)
@@ -1,4 +1,4 @@
 <?xml version="1.0"?>
-<robot name="starsthing" xmlns:xacro="http://ros.org/wiki/xacro" >
+<robot name="UR5_2F85" xmlns:xacro="http://ros.org/wiki/xacro" >
 	<!-- On the first day, Darwin created the world -->
     <link name="world"/>
@@ -20,7 +20,18 @@
   	/>
 	<!-- Add Robotiq 2f-85 gripper -->
-    <xacro:include filename="./robotiq_2f_model/robotiq_2f_85.urdf.xacro" />
-	<xacro:robotiq_2f_85 parent="ee_link" name="gripper" precise_collision="true" adaptive_transmission="true" with_pads="true" >
-		<origin xyz="0 0 0" rpy="0 ${pi/2} 0"/>
-	</xacro:robotiq_2f_85>
+    <xacro:include filename="./Robotiq_2F85/urdf/Robotiq_2F85.urdf.xacro" />
+	<xacro:Robotiq_2F85 parent="ee_link" name="gripper" enable_underactuation="true" soft_pads="true" softness="5" >
+		<origin xyz="0 0 0" rpy="0 0 ${pi/2}"/>
+	</xacro:Robotiq_2F85>
+    <!-- Add a Tool Center Point reference as a convenience.
+         The TCP is at 18.75mm from the tip of the gripper as its located in
+         the middle of the pad. As a result, if the TCP is at 18.75mm above the floor,
+         it means that the gripper touches the floor. If you want the TCP to
+         be located at the tip of the gripper, use 0.14948 instead of 0.13073 -->
+    <joint name="tool_center_point" type="fixed">
+        <origin rpy="${pi/2} ${pi/2} 0" xyz="0 -0.14948 0"/>
+        <parent link="gripper_base"/>
+        <child link="tcp"/>
+    </joint>
+    <link name="tcp" />
 </robot>
