Commit message: Modified fictious links with undefined inertial parameters.

File: models/UR5.urdf (robot description, URDF)
Before this commit: robot UR5, 10 links, 9 joints
Links:
- link base: mass None -> 0
- link ee_link: mass None -> 0

File: models/UR5_2F85.urdf (robot description, URDF)
Before this commit: robot UR5_2F85, 22 links, 21 joints
Links:
- link base: mass None -> 0
- link ee_link: mass None -> 0
- link tcp: mass None -> 0

File: models/UR5_2F85_BuildURDF.xacro (robot description, xacro)
@@ -34,4 +34,10 @@
         <child link="tcp"/>
     </joint>
-    <link name="tcp" />
+    <link name="tcp" >
+        <!-- If no inertial parameters are supplied, PyBullet will use a mass of 1Kg. -->
+        <inertial>
+            <mass value="0"/>
+            <inertia ixx="0.0" ixy="0.0" ixz="0.0" iyy="0.0" iyz="0.0" izz="0.0"/>
+        </inertial>
+    </link>
 </robot>

File: models/ur5/ur5.urdf.xacro (robot description, xacro)
@@ -329,9 +329,18 @@
         <origin rpy="0 0 0" xyz="-0.01 0 0"/>
       </collision>
+      <inertial>
+        <mass value="0"/>
+        <inertia ixx="0.0" ixy="0.0" ixz="0.0" iyy="0.0" iyz="0.0" izz="0.0"/>
+      </inertial>
     </link>
     <!-- <xacro:ur_arm_transmission prefix="${prefix}" hw_interface="${transmission_hw_interface}" /> -->
     <!-- <xacro:ur_arm_gazebo prefix="${prefix}" /> -->
     <!-- ROS base_link to UR 'Base' Coordinates transform -->
-    <link name="${prefix}base"/>
+    <link name="${prefix}base">
+      <inertial>
+        <mass value="0"/>
+        <inertia ixx="0.0" ixy="0.0" ixz="0.0" iyy="0.0" iyz="0.0" izz="0.0"/>
+      </inertial>
+    </link>
     <joint name="${prefix}base_link-base_fixed_joint" type="fixed">
       <!-- NOTE: this rotation is only needed as long as base_link itself is
