Commit message: Removed forgotten hardcoded gripper name

File: pbsm/models/Robotiq_2F85/urdf/Robotiq_2F85.urdf.xacro (robot description, xacro)
@@ -341,7 +341,7 @@
       rpy="3.1416 0 -2.9033" />
     <parent
-      link="gripper_right_coupler" />
-    <child
-      link="gripper_right_follower" />
+      link="${name}_right_coupler" />
+    <child
+      link="${name}_right_follower" />
     <axis
       xyz="0 0 1" />
